File: THE SPLITY/THE SPLITY.kicad_pcb (KiCad board)
At the start: 2 copper layers, 139.3 x 108.3 mm, 59 parts, among them U2 Nice_Nano_V2

Commit message: goo gaga
Routing:
- added copper zone on B.Cu, net (none)
- added copper zone on F.Cu, net (none)
Changed lines of the file:
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@@
 		(net 40)
+	)
+	(zone
+		(net 0)
+		(net_name "")
+		(layers "F.Cu" "B.Cu")
+		(hatch edge 0.5)
+		(connect_pads
+			(clearance 0.5)
+		)
+		(min_thickness 0.25)
+		(filled_areas_thickness no)
+		(fill yes
+			(thermal_gap 0.5)
+			(thermal_bridge_width 0.5)
+			(island_removal_mode 1)
+			(island_area_min 10)
+		)
+		(polygon
+			(pts
+				(xy 131 39) (xy 146 165) (xy 379 161.5) (xy 374.5 29) (xy 131 39.5)
+			)
+		)
 	)
 	(embedded_fonts no)
