File: THE SPLITY/THE SPLITY.kicad_pcb (KiCad board)
At the start: 2 copper layers, 139.3 x 108.3 mm, 59 parts, among them U2 Nice_Nano_V2

Commit message: added a battery connector
boo
Parts:
- added J1: Conn_01x02_Socket, Connector_JST:JST_XH_B2B-XH-AM_1x02_P2.50mm_Vertical, B.Cu at (177.8, 124.5)
Connections:
- U2 pad 23: unconnected-(U2-GND-Pad23) -> -
- U2 pad 24: unconnected-(U2-B+-Pad24) -> +
Routing:
- net +: track 0.00 -> 68.8 mm
- net -: track 0.00 -> 66.5 mm
