File: THE SPLITY/THE SPLITY.kicad_pcb (KiCad board)
At the start: 2 copper layers, 139.3 x 108.3 mm, 60 parts, among them J1 Conn_01x02_Socket, U2 Nice_Nano_V2

Commit message: ז
Parts:
- added SW1: Switch, ScottoKeebs_Components:Switch_K3-1204D, F.Cu at (5.05, 1.30)
Connections:
- U2 pad 22: unconnected-(U2-RST-Pad22) -> RST
- U2 pad 23: - -> GND
Changed lines of the file:
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@@
 	(net 47 "unconnected-(U2-0-Pad2)")
 	(net 48 "-")
-	(net 49 "unconnected-(U2-RST-Pad22)")
+	(net 49 "GND")
 	(net 50 "unconnected-(U2-Pad1)")
 	(net 51 "unconnected-(U2-1-Pad25)")
@@
 	(net 55 "unconnected-(U2-20-Pad19)")
 	(net 56 "unconnected-(U2-19-Pad18)")
+	(net 57 "RST")
 	(footprint "ScottoKeebs_MX:MX_PCB_1.00u"
 		(layer "F.Cu")
@@
 			(layers "*.Cu" "*.Mask")
 			(remove_unused_layers no)
-			(net 49 "unconnected-(U2-RST-Pad22)")
+			(net 57 "RST")
 			(pinfunction "RST")
 			(pintype "input")
@@
 			(layers "*.Cu" "*.Mask")
 			(remove_unused_layers no)
-			(net 48 "-")
+			(net 49 "GND")
 			(pinfunction "GND")
 			(pintype "input")
@@
 		)
 	)
+	(footprint "ScottoKeebs_Components:Switch_K3-1204D"
+		(layer "F.Cu")
+		(at 5.05 1.3)
+		(property "Reference" "SW1"
+			(at 0 -0.5 0)
+			(unlocked yes)
+			(layer "F.SilkS")
+			(hide yes)
+			(effects
+				(font
+					(size 1 1)
+					(thickness 0.1)
+				)
+			)
+		)
+		(property "Value" "Switch"
+			(at 0 1 0)
+			(unlocked yes)
+			(layer "F.Fab")
+			(hide yes)
+			(effects
+				(font
+					(size 1 1)
+					(thickness 0.15)
+				)
+			)
+		)
+		(property "Datasheet" "~"
+			(at 0 0 0)
+			(unlocked yes)
+			(layer "F.Fab")
+			(hide yes)
+			(effects
+				(font
+					(size 1 1)
+					(thickness 0.15)
+				)
+			)
+		)
+		(property "Description" "Push button switch, generic, two pins"
+			(at 0 0 0)
+			(unlocked yes)
+			(layer "F.Fab")
+			(hide yes)
+			(effects
+				(font
+					(size 1 1)
+					(thickness 0.15)
+				)
+			)
+		)
+		(property "LCSC" "C145861"
+			(at 0 -3 0)
+			(unlocked yes)
+			(layer "F.SilkS")
+			(hide yes)
+			(effects
+				(font
+					(size 1 1)
+					(thickness 0.1)
+				)
+			)
+		)
+		(sheetname "/")
+		(sheetfile "THE SPLITY.kicad_sch")
+		(attr through_hole)
+		(fp_rect
+			(start -5 -1.25)
+			(end 5 1.25)
+			(stroke
+				(width 0.1)
+				(type default)
+			)
+			(fill no)
+			(layer "Dwgs.User")
+		)
+		(fp_rect
+			(start -5 -1.25)
+			(end 5 1.25)
+			(stroke
+				(width 0.1)
+				(type default)
+			)
+			(fill no)
+			(layer "F.CrtYd")
+		)
+		(pad "1" thru_hole circle
+			(at -2.55 0)
+			(size 1.524 1.524)
+			(drill 0.762)
+			(layers "*.Cu" "*.Mask")
+			(remove_unused_layers no)
+			(net 49 "GND")
+			(pinfunction "1")
+			(pintype "passive")
+		)
+		(pad "2" thru_hole circle
+			(at 0 0)
+			(size 1.524 1.524)
+			(drill 0.762)
+			(layers "*.Cu" "*.Mask")
+			(remove_unused_layers no)
+			(net 48 "-")
+			(pinfunction "2")
+			(pintype "passive")
+		)
+		(pad "3" thru_hole circle
+			(at 2.55 0)
+			(size 1.524 1.524)
+			(drill 0.762)
+			(layers "*.Cu" "*.Mask")
+			(remove_unused_layers no)
+		)
+		(embedded_fonts no)
+	)
 	(footprint "ScottoKeebs_MX:MX_PCB_1.00u"

Commit message: mounting holes and outline change
Parts:
- removed SW1: Switch, ScottoKeebs_Components:Switch_K3-1204D
- added H1: MountingHole, MountingHole:MountingHole_2.2mm_M2, F.Cu at (290.5, 111.9)
- added H2: MountingHole, MountingHole:MountingHole_2.2mm_M2, F.Cu at (190.5, 122.6)
- added H3: MountingHole, MountingHole:MountingHole_2.2mm_M2, F.Cu at (233.4, 67.9)
- added H4: MountingHole, MountingHole:MountingHole_2.2mm_M2, F.Cu at (289.3, 92.9)
- added H5: MountingHole, MountingHole:MountingHole_2.2mm_M2, F.Cu at (197.6, 71.4)
- added H6: MountingHole, MountingHole:MountingHole_2.2mm_M2, F.Cu at (233.4, 106.0)
Connections:
- U2 pad 22: RST -> unconnected-(U2-RST-Pad22)
- U2 pad 23: GND -> -
Routing:
- net column 3: track 257.9 -> 268.9 mm
- net column 5: track 277.4 -> 276.5 mm
- net column 4: track 258.0 -> 257.0 mm
- net -: track 66.5 -> 67.3 mm
Other:
- outline, holes or cut-outs redrawn

Commit message: z
Parts:
- added H2: MountingHole, MountingHole:MountingHole_2.2mm_M2, F.Cu at (178.6, 119.1)
- moved H2 29.0 mm to (219.1, 127.4)
- moved J1 1.88 mm to (178.6, 126.2), turned to -90 degrees
Routing:
- net -: track 67.3 -> 76.6 mm
- net +: track 68.8 -> 70.8 mm

Commit message: updated some stuff
Other:
- board size 139.3 x 108.3 mm -> 307.2 x 108.3 mm
