File: THE SPLITY/v2 pcb/THE 58 V2/THE 58 V2.kicad_pcb (KiCad board)
At the start: 2 copper layers, 137 parts, among them J1 Conn_01x02_Socket, J2 Conn_01x02_Socket, SW1 Switch, U1 Nice_Nano_V2, U2 Nice_Nano_V2, U3 TRRS, U4 TRRS

Commit message: updated schem
Parts:
- added SW2: Switch, ScottoKeebs_Components:Button_MJTP1243, F.Cu at (158.8, 152.7)
- added SW3: Switch, ScottoKeebs_Components:Switch_MSK12C02, F.Cu at (158.6, 138.4)
- added SW4: Switch, ScottoKeebs_Components:Button_MJTP1243, F.Cu at (158.8, 157.7)
- S1, S10, S11, S12, S13, S14, S15, S16, S17, S18, S19, S2, S20, S21, S22, S23, S24, S25, S26, S27, S28, S29, S3, S30, S31, S32, S33, S34, S35, S36, S37, S38, S39, S4, S40, S41, S42, S43, S44, S45, S46, S47, S48, S49, S5, S50, S51, S52, S53, S54, S55, S56, S57, S58, S6, S7, S8, S9: footprint ScottoKeebs_MX:MX_PCB_1.00u -> ScottoKeebs_MX:MX_PCB_1.00u_Reversable
- moved S8 263.0 mm to (280.0, 62.2)
- moved S2 239.5 mm to (256.9, 59.7)
- moved S1 222.2 mm to (237.8, 61.9)
- moved S3 171.5 mm to (189.5, 57.5)
- moved J1 117.8 mm to (150.9, 153.5)
- moved J2 117.8 mm to (150.9, 161.3)
- moved H1 117.8 mm to (126.6, 153.1)
- moved H2 117.8 mm to (126.6, 159.1)
- moved H3 117.8 mm to (126.6, 165.0)
- moved H7 117.8 mm to (138.5, 153.1)
- moved H8 117.8 mm to (138.5, 159.1)
- moved H9 117.8 mm to (138.5, 165.0)
- moved H10 117.8 mm to (144.5, 153.1)
- moved H11 117.8 mm to (144.5, 159.1)
- moved H12 117.8 mm to (144.5, 165.0)
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Connections:
- J2 pad 2: -. -> gnd.
- S30 pad 1: column 0. -> column -1.
- U1 pad 1: unconnected-(U1-Pad1) -> cs.
- U1 pad 10: column 5. -> unconnected-(U1-7-Pad10)
- U1 pad 13: row 4. -> unconnected-(U1-10-Pad13)
- U1 pad 14: row 3. -> unconnected-(U1-16-Pad14)
- U1 pad 15: row 2. -> unconnected-(U1-14-Pad15)
- U1 pad 16: row 1. -> unconnected-(U1-15-Pad16)
- U1 pad 17: row 0. -> unconnected-(U1-18-Pad17)
- U1 pad 2: unconnected-(U1-0-Pad2) -> 19.
- U1 pad 20: 20. -> unconnected-(U1-21-Pad20)
- U1 pad 22: unconnected-(U1-RST-Pad22) -> rst.
- U1 pad 23: -. -> unconnected-(U1-GND-Pad23)
- U1 pad 24: +. -> b+.
- U1 pad 3: unconnected-(U1-GND-Pad3) -> -.
- U1 pad 4: gnd. -> unconnected-(U1-GND-Pad4)
- U1 pad 5: column 0. -> mosi.
- U1 pad 6: column 1. -> sck.
- U1 pad 7: column 2. -> 20.
- U1 pad 8: column 3. -> unconnected-(U1-5-Pad8)
- U1 pad 9: column 4. -> unconnected-(U1-6-Pad9)
- U2 pad 22: unconnected-(U2-RST-Pad22) -> rst
- U2 pad 3: gnd -> -
- U4 pad 4: unconnected-(U4-RING2-Pad4) -> 19.

Commit message: almost half way done pcb
Parts:
- added D59: Diode, ScottoKeebs_Components:Diode_DO-35, F.Cu at (246.5, 139.5)
- added D60: Diode, ScottoKeebs_Components:Diode_DO-35, F.Cu at (-14.2, 117.5)
- added S59: Keyswitch, ScottoKeebs_MX:MX_PCB_1.00u, F.Cu at (236.9, 135.7)
- added S60: Keyswitch, ScottoKeebs_MX:MX_PCB_1.00u_Reversable, F.Cu at (-7.99, 107.9)
- J1: moved to B.Cu
- S1, S10, S11, S12, S13, S14, S15, S16, S17, S18, S19, S2, S20, S21, S22, S23, S24, S25, S26, S27, S28, S29, S3, S30, S31, S32, S33, S34, S35, S36, S37, S38, S39, S4, S40, S41, S42, S43, S44, S45, S46, S47, S48, S49, S5, S50, S51, S52, S53, S54, S55, S56, S57, S58, S6, S7, S8, S9: footprint ScottoKeebs_MX:MX_PCB_1.00u_Reversable -> ScottoKeebs_MX:MX_PCB_1.00u
- moved S6 314.3 mm to (333.4, 64.3)
- moved S18 300.3 mm to (333.4, 102.4)
- moved S12 295.9 mm to (333.4, 83.3)
- moved S5 293.7 mm to (314.3, 61.9)
- moved S24 279.9 mm to (333.4, 121.4)
- moved S17 279.4 mm to (314.3, 100.0)
- moved S11 278.1 mm to (314.3, 81.0)
- moved S4 273.6 mm to (295.3, 57.1)
- moved S9 267.1 mm to (276.2, 73.8)
- moved S23 261.7 mm to (314.3, 119.1)
- moved S10 260.7 mm to (295.3, 76.2)
- moved S16 259.0 mm to (295.3, 95.2)
- moved S22 244.1 mm to (295.3, 114.3)
- moved S26 240.6 mm to (294.1, 133.3)
- moved S15 238.8 mm to (276.2, 92.9)
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Connections:
- S29 pad 1: column 0 -> column -1
- S31 pad 1: column 0. -> column -1.
Routing:
- net row 2: track 0.00 -> 113.9 mm
- net vcc: track 0.00 -> 93.3 mm
- net row 1: track 0.00 -> 91.6 mm
- net row 0: track 0.00 -> 91.6 mm
- net row 3: track 0.00 -> 91.6 mm
- net column 2: track 0.00 -> 89.3 mm
- net 19: track 0.00 -> 88.6 mm
- net column 3: track 0.00 -> 86.6 mm
- net column 4: track 0.00 -> 84.4 mm
- net 20: track 0.00 -> 78.3 mm
- net column 0: track 0.00 -> 76.7 mm
- net row 4: track 0.00 -> 75.7 mm
- net b+: track 0.00 -> 73.8 mm, vias 0 -> 1
- net column 5: track 0.00 -> 59.9 mm
- net gnd: track 0.00 -> 58.3 mm
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
Commit message: almost finished the pcb
Parts:
- added H13: MountingHole, MountingHole:MountingHole_2.2mm_M2, F.Cu at (184.6, 60.4)
- added H14: MountingHole, MountingHole:MountingHole_2.2mm_M2, F.Cu at (184.5, 66.7)
- added H15: MountingHole, MountingHole:MountingHole_2.2mm_M2, F.Cu at (184.5, 72.6)
- added H16: MountingHole, MountingHole:MountingHole_2.2mm_M2, F.Cu at (184.5, 78.6)
- added R1: Resistor, Resistor_THT:R_Axial_DIN0207_L6.3mm_D2.5mm_P7.62mm_Horizontal, F.Cu at (226.2, 93.1)
- added R2: Resistor, Resistor_THT:R_Axial_DIN0207_L6.3mm_D2.5mm_P7.62mm_Horizontal, F.Cu at (138.1, 93.1)
- J2: moved to B.Cu
- S60: footprint ScottoKeebs_MX:MX_PCB_1.00u_Reversable -> ScottoKeebs_MX:MX_PCB_1.00u
- moved H7 203.7 mm to (303.6, 127.4)
- moved S31 147.7 mm to (148.8, 139.3), turned to -15 degrees
- moved D57 146.2 mm to (34.8, 111.9), turned to 180 degrees
- moved D54 144.3 mm to (40.5, 122.9)
- moved D45 138.7 mm to (79.8, 138.4)
- moved S60 138.2 mm to (127.4, 135.7)
- moved D58 134.2 mm to (53.8, 109.5), turned to 180 degrees
- moved D60 133.9 mm to (117.9, 139.5), turned to 90 degrees
- moved S30 133.5 mm to (145.3, 103.6)
- moved D56 130.4 mm to (34.8, 92.9), turned to 180 degrees
- moved D31 130.1 mm to (138.3, 139.4), turned to 75 degrees
- moved D53 127.0 mm to (40.5, 103.8)
- moved D40 126.6 mm to (98.8, 139.5)
- moved D50 123.7 mm to (74.1, 123.8), turned to 180 degrees
- moved H6 123.5 mm to (216.7, 122.6)
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Connections:
- U1 pad 10: unconnected-(U1-7-Pad10) -> column 0.
- U1 pad 11: unconnected-(U1-8-Pad11) -> column -1.
- U1 pad 13: unconnected-(U1-10-Pad13) -> column 3.
- U1 pad 14: unconnected-(U1-16-Pad14) -> column 4.
- U1 pad 15: unconnected-(U1-14-Pad15) -> column 5.
- U1 pad 16: unconnected-(U1-15-Pad16) -> row 4.
- U1 pad 17: unconnected-(U1-18-Pad17) -> row 3.
- U1 pad 18: unconnected-(U1-19-Pad18) -> row 2.
- U1 pad 19: unconnected-(U1-20-Pad19) -> row 1.
- U1 pad 20: unconnected-(U1-21-Pad20) -> row 0.
- U1 pad 25: cs. -> unconnected-(U1-1-Pad25)
- U1 pad 26: sck. -> unconnected-(U1-2-Pad26)
- U1 pad 27: mosi. -> unconnected-(U1-7-Pad27)
- U1 pad 8: unconnected-(U1-5-Pad8) -> column 2.
- U1 pad 9: unconnected-(U1-6-Pad9) -> column 1.
- U2 pad 10: unconnected-(U2-7-Pad10) -> column 0
- U2 pad 11: unconnected-(U2-8-Pad11) -> column -1
- U2 pad 13: unconnected-(U2-10-Pad13) -> column 5
- U2 pad 14: unconnected-(U2-16-Pad14) -> column 4
- U2 pad 15: unconnected-(U2-14-Pad15) -> column 3
- U2 pad 16: unconnected-(U2-15-Pad16) -> row 0
- U2 pad 17: unconnected-(U2-18-Pad17) -> row 1
- U2 pad 18: unconnected-(U2-19-Pad18) -> row 2
- U2 pad 19: unconnected-(U2-20-Pad19) -> row 3
- U2 pad 20: unconnected-(U2-21-Pad20) -> row 4
- U2 pad 8: unconnected-(U2-5-Pad8) -> column 2
- U2 pad 9: unconnected-(U2-6-Pad9) -> column 1
Routing:
- net row 0.: track 0.00 -> 279.8 mm
- net row 1.: track 0.00 -> 259.1 mm
- net row 2.: track 0.00 -> 259.1 mm
- net column 2.: track 0.00 -> 229.2 mm
- net column 4.: track 0.00 -> 225.4 mm
- net column 5.: track 0.00 -> 215.9 mm
- net row 3.: track 0.00 -> 215.0 mm
- net column 3.: track 0.00 -> 204.2 mm
- net row 0: track 91.6 -> 287.7 mm
- net row 1: track 91.6 -> 272.5 mm
- net column 5: track 59.9 -> 235.8 mm, vias 0 -> 1
- net column 1.: track 0.00 -> 170.9 mm
- net row 3: track 91.6 -> 255.8 mm
- net column 0.: track 0.00 -> 161.7 mm
- net column 4: track 84.4 -> 237.2 mm, vias 0 -> 1
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Other:
- board outline added: 323.8 x 107.7 mm
