File: THE SPLITY/v2 pcb/THE 58 V2/THE 58 V2.kicad_sch (KiCad schematic)
At the start: 136 parts, among them J1 Conn_01x02_Socket, J2 Conn_01x02_Socket, U1 Nice_Nano_V2, U2 Nice_Nano_V2, U3 TRRS, U4 TRRS

Commit message: v2
Parts:
- added SW1: Switch, ScottoKeebs_Components:Switch_MSK12C02, symbol ScottoKeebs:Placeholder_Switch
- Display1, Display2: footprint nice_view:nice_view -> nice view:nice_view
Connections:
- net +: now also SW1.2; no longer U2.24 (B+)
- net 20: now also U2.7 (4); no longer U2.20 (21)
- net column 0: no longer S25.1, U2.5 (2)
- net column 1: no longer U2.6 (3)
- net column 2: no longer U2.7 (4)
- net column 3: no longer U2.8 (5)
- net column 4: no longer U2.9 (6)
- net column 5: no longer U2.10 (7)
- net cs: now also U2.1; no longer U2.25 (1)
- net gnd: now also J1.2 (Pin_2), U2.3 (GND); no longer U2.4 (GND)
- net mosi: now also U2.5 (2); no longer U2.27 (7)
- net row 0: no longer U2.17 (18)
- net row 1: no longer U2.16 (15)
- net row 2: no longer U2.15 (14)
- net row 3: no longer U2.14 (16)
- net row 4: no longer U2.13 (10)
- net sck: now also U2.6 (3); no longer U2.26 (2)
- net 19: now reaches U3.4 (RING2)
- net 19: now also U2.2 (0)
- net -: no longer names the net of U2.23 (GND)
- net -: no longer J1.2 (Pin_2)
- new net b+: SW1.1, U2.24 (B+)
- new net column -1: S25.1
Other:
- moved on the sheet: Display1, J1

Commit message: updated schem
Parts:
- added R1, R2: Resistor, symbol ScottoKeebs:Placeholder_Resistor
- added SW2, SW4: Switch, ScottoKeebs_Components:Button_MJTP1243, symbol ScottoKeebs:Placeholder_Switch
- added SW3: Switch, ScottoKeebs_Components:Switch_MSK12C02, symbol ScottoKeebs:Placeholder_Switch
- S1, S10, S11, S12, S13, S14, S15, S16, S17, S18, S19, S2, S20, S21, S22, S23, S24, S25, S26, S27, S28, S29, S3, S30, S31, S32, S33, S34, S35, S36, S37, S38, S39, S4, S40, S41, S42, S43, S44, S45, S46, S47, S48, S49, S5, S50, S51, S52, S53, S54, S55, S56, S57, S58, S6, S7, S8, S9: footprint ScottoKeebs_MX:MX_PCB_1.00u -> ScottoKeebs_MX:MX_PCB_1.00u_Reversable
Connections:
- net +.: now also SW3.2; no longer U1.24 (B+)
- net -.: now also U1.3 (GND), R2.2; no longer J2.2 (Pin_2), U1.23 (GND)
- net 20.: now also U1.7 (4); no longer U1.20 (21)
- net column 0.: no longer S30.1, U1.5 (2)
- net column 1.: no longer U1.6 (3)
- net column 2.: no longer U1.7 (4)
- net column 3.: no longer U1.8 (5)
- net column 4.: no longer U1.9 (6)
- net column 5.: no longer U1.10 (7)
- net cs.: now also U1.1
- net gnd: now also R1.1, SW2.2; no longer U2.3 (GND)
- net gnd.: now also J2.2 (Pin_2), R2.1, SW4.2; no longer U1.4 (GND)
- net mosi.: now also U1.5 (2)
- net row 0.: no longer U1.17 (18)
- net row 1.: no longer U1.16 (15)
- net row 2.: no longer U1.15 (14)
- net row 3.: no longer U1.14 (16)
- net row 4.: no longer U1.13 (10)
- net sck.: now also U1.6 (3)
- net 19.: now reaches U4.4 (RING2)
- net 19.: now also U1.2 (0)
- net rst: now reaches U2.22 (RST)
- net rst: now also SW2.1
- net rst.: now reaches U1.22 (RST)
- net rst.: now also SW4.1
- new net -: R1.2, U2.3 (GND)
- new net b+.: SW3.1, U1.24 (B+)
- new net column -1.: S30.1
Other:
- moved on the sheet: U2, U4

Commit message: almost half way done pcb
Parts:
- added D59, D60: Diode, ScottoKeebs_Components:Diode_DO-35, symbol ScottoKeebs:Placeholder_Diode
- added S59: Keyswitch, ScottoKeebs_MX:MX_PCB_1.00u, symbol ScottoKeebs:Placeholder_Keyswitch
- added S60: Keyswitch, ScottoKeebs_MX:MX_PCB_1.00u_Reversable, symbol ScottoKeebs:Placeholder_Keyswitch
- S1, S10, S11, S12, S13, S14, S15, S16, S17, S18, S19, S2, S20, S21, S22, S23, S24, S25, S26, S27, S28, S29, S3, S30, S31, S32, S33, S34, S35, S36, S37, S38, S39, S4, S40, S41, S42, S43, S44, S45, S46, S47, S48, S49, S5, S50, S51, S52, S53, S54, S55, S56, S57, S58, S6, S7, S8, S9: footprint ScottoKeebs_MX:MX_PCB_1.00u_Reversable -> ScottoKeebs_MX:MX_PCB_1.00u
Connections:
- net column -1: now also S29.1
- net column -1.: now also S31.1
- net column 0: now also S59.1; no longer S29.1
- net column 0.: now also S60.1; no longer S31.1
- net row 4: now also D59.1 (K)
- net row 4.: now also D60.1 (K)
- new net: D59.2 (A), S59.2
- new net: D60.2 (A), S60.2
Other:
- moved on the sheet: D29, D31, S29, S31

Commit message: almost finished the pcb
Parts:
- added H13, H14, H15, H16: MountingHole, MountingHole:MountingHole_2.2mm_M2, symbol Mechanical:MountingHole
- R1, R2: footprint (none) -> Resistor_THT:R_Axial_DIN0207_L6.3mm_D2.5mm_P7.62mm_Horizontal
- S60: footprint ScottoKeebs_MX:MX_PCB_1.00u_Reversable -> ScottoKeebs_MX:MX_PCB_1.00u
Connections:
- net -: now also R1.1; no longer R1.2
- net column -1: now also U2.11 (8)
- net column -1.: now also U1.11 (8)
- net column 0: now also U2.10 (7)
- net column 0.: now also U1.10 (7)
- net column 1: now also U2.9 (6)
- net column 1.: now also U1.9 (6)
- net column 2: now also U2.8 (5)
- net column 2.: now also U1.8 (5)
- net column 3: now also U2.15 (14)
- net column 3.: now also U1.13 (10)
- net column 4: now also U2.14 (16)
- net column 4.: now also U1.14 (16)
- net column 5: now also U2.13 (10)
- net column 5.: now also U1.15 (14)
- net cs.: no longer U1.25 (1)
- net gnd: now also R1.2; no longer R1.1
- net mosi.: no longer U1.27 (7)
- net row 0: now also U2.16 (15)
- net row 0.: now also U1.20 (21)
- net row 1: now also U2.17 (18)
- net row 1.: now also U1.19 (20)
- net row 2: now also U2.18 (19)
- net row 2.: now also U1.18 (19)
- net row 3: now also U2.19 (20)
- net row 3.: now also U1.17 (18)
- net row 4: now also U2.20 (21)
- net row 4.: now also U1.16 (15)
- net sck.: no longer U1.26 (2)
Other:
- moved on the sheet: R1
