File: THE 60/v2 pcb/THE 60 V2/THE 58 V2.kicad_pcb (KiCad board)
At the start: 2 copper layers, 323.8 x 107.7 mm, 136 parts, among them J1 Conn_01x02_Socket, J2 Conn_01x02_Socket, SW1 Switch, SW2 Switch, SW3 Switch, SW4 Switch, U1 Nice_Nano_V2, U2 Nice_Nano_V2, U3 TRRS, U4 TRRS

Commit message: added silk screen
Parts:
- added G***: LOGO, logoo:hedwig rightttt, F.Cu at (119.1, 92.9)
- added G***: LOGO, logoo:hedwig leftttt, F.Cu at (245.3, 92.9)

Commit message: another silk screen
Parts:
- added G***: LOGO, logoo:hogwarts, F.Cu at (216.7, 60.7)
- added G***: LOGO, logoo:hogwarts, F.Cu at (147.6, 60.7)
- turned S40 to 0 degrees
Other:
- board text added: "made by me :)"
- board text added: "you can find me in github: eyalbirger"
