File: THE 60/v2 pcb/THE 60 V2/THE 58 V2.kicad_pcb (KiCad board)
At the start: 2 copper layers, 323.8 x 107.7 mm, 140 parts, among them J1 Conn_01x02_Socket, J2 Conn_01x02_Socket, SW1 Switch, SW2 Switch, SW3 Switch, SW4 Switch, U1 Nice_Nano_V2, U2 Nice_Nano_V2, U3 TRRS, U4 TRRS

Commit message: z
Parts:
- moved G*** 1.19 mm to (244.1, 92.9)
Connections:
- J1 pad 1: + -> gnd
- J1 pad 2: gnd -> +
- J2 pad 1: +. -> gnd.
- J2 pad 2: gnd. -> +.
Routing:
- net +.: track 16.8 -> 14.3 mm
- net gnd.: track 75.1 -> 76.9 mm
- net row 3: track 253.0 -> 251.5 mm
- net row 1: track 277.1 -> 275.5 mm
- net row 0: track 291.0 -> 289.4 mm
- net row 4: track 189.8 -> 188.3 mm
- net gnd: track 69.6 -> 68.1 mm
- net +: track 10.9 -> 10.0 mm
Other:
- board size 323.8 x 107.7 mm -> 323.8 x 107.2 mm
- board text added: "+"
- board text added: "-"

Commit message: Panelized it
Parts:
- moved D11 176.4 mm to (147.6, 76.4)
- moved D17 176.4 mm to (147.6, 95.5)
- moved D23 176.4 mm to (147.6, 114.5)
- moved D26 176.4 mm to (114.1, 115.5)
- moved D5 176.4 mm to (147.6, 57.4)
- moved S15 176.4 mm to (100.0, 84.5)
- moved S21 176.4 mm to (100.0, 103.6)
- moved S26 176.4 mm to (117.9, 125.0)
- moved S3 176.4 mm to (100.0, 46.4)
- moved S9 176.4 mm to (100.0, 65.5)
- moved D1 176.4 mm to (71.4, 55.0)
- moved D10 176.4 mm to (128.6, 72.9)
- moved D12 176.4 mm to (153.4, 84.5)
- moved D13 176.4 mm to (71.4, 93.1)
- moved D15 176.4 mm to (109.5, 88.3)
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Other:
- board size 323.8 x 107.2 mm -> 284.6 x 107.2 mm
- board text added: "{dblquote}Dobby is free{dblquote}"
- board text added: "{dblquote}help will always be given at hogwarts to those who deserve it{dblquote}"

Commit message: /
Other:
- board text added: "Dobby is free"
- board text removed: "{dblquote}Dobby is free{dblquote}"
