File: THE 60/v2 pcb/THE 60 V2/THE 58 V2.kicad_pcb (KiCad board)
At the start: 2 copper layers, 284.6 x 107.2 mm, 140 parts, among them J1 Conn_01x02_Socket, J2 Conn_01x02_Socket, SW1 Switch, SW2 Switch, SW3 Switch, SW4 Switch, U1 Nice_Nano_V2, U2 Nice_Nano_V2, U3 TRRS, U4 TRRS

Commit message: /
/
Parts:
- moved H12 68.6 mm to (331.6, 173.2)
- moved J2 68.6 mm to (325.6, 175.7)
- moved S43 68.6 mm to (272.1, 143.5)
- moved D10 68.6 mm to (163.7, 131.8)
- moved D12 68.6 mm to (188.5, 143.5)
- moved D23 68.6 mm to (182.8, 173.5)
- moved D3 68.6 mm to (144.7, 109.2)
- moved D30 68.6 mm to (319.7, 158.0)
- moved D34 68.6 mm to (300.6, 152.0)
- moved D37 68.6 mm to (281.6, 131.8)
- moved D47 68.6 mm to (243.5, 131.8)
- moved D50 68.6 mm to (258.0, 174.4)
- moved D54 68.6 mm to (224.4, 173.5)
- moved D60 68.6 mm to (301.8, 190.1)
- moved D8 68.6 mm to (125.6, 131.8)
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Routing:
- net b+.: track 91.1 -> 96.9 mm
- net vcc.: track 86.8 -> 92.0 mm
- net gnd.: track 76.9 -> 79.1 mm
- net rst.: track 40.9 -> 39.5 mm
Other:
- outline, holes or cut-outs redrawn
- board text added: "{dblquote}It is our choices, Harry, that show what we truly are, far more than our abilities.{dblquote}"

Commit message: finally finished this
Parts:
- added D61: LED, custom:pad - oval2.5x1.5, B.Cu at (80.4, 104.2)
- added D62: LED, custom:pad - oval2.5x1.5, B.Cu at (70.8, 104.2)
- added D63: LED, custom:pad - oval2.5x1.5, B.Cu at (326.8, 104.2)
- added D64: LED, custom:pad - oval2.5x1.5, B.Cu at (336.3, 104.2)
- added G***: LOGO, logoo:the deathly hallows symbol, F.Cu at (220.9, 178.6)
- added G***: LOGO, logoo:the deathly hallows symbol, F.Cu at (186.9, 178.6)
Routing:
- net row 1.: track 262.2 -> 123.6 mm
- net row 0: track 289.4 -> 165.5 mm
- net row 2.: track 261.0 -> 156.9 mm
- net +: track 10.0 -> 110.8 mm
- net +.: track 14.3 -> 110.9 mm, vias 1 -> 2
- net row 1: track 275.5 -> 182.3 mm
- net row 3.: track 217.3 -> 157.3 mm, vias 0 -> 1
- net gnd: track 68.1 -> 123.6 mm, vias 1 -> 2
- net column 2.: track 232.7 -> 188.6 mm, vias 0 -> 2
- net row 0.: track 284.5 -> 240.4 mm, vias 0 -> 1
- net gnd.: track 79.1 -> 115.8 mm
- net column -1.: track 110.0 -> 74.1 mm
- net column 0.: track 160.2 -> 192.0 mm
- net column 1.: track 170.5 -> 140.2 mm
- net vcc.: track 92.0 -> 67.3 mm, vias 1 -> 0
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