File: THE 60/v2 pcb/THE 60 V2/THE 58 V2.kicad_sch (KiCad schematic)
At the start: 150 parts, among them J1 Conn_01x02_Socket, J2 Conn_01x02_Socket, SW1 Switch, SW2 Switch, SW3 Switch, SW4 Switch, U1 Nice_Nano_V2, U2 Nice_Nano_V2, U3 TRRS, U4 TRRS

Commit message: added silk screen
Parts:
- removed H1, H10, H11, H13, H14, H15, H16, H2, H3, H4, H5, H7, H8, H9: MountingHole, MountingHole:MountingHole_2.2mm_M2, symbol Mechanical:MountingHole

Commit message: z
Connections:
- net +: now also J1.2 (Pin_2); no longer J1.1 (Pin_1)
- net +.: now also J2.2 (Pin_2); no longer J2.1 (Pin_1)
- net gnd: now also J1.1 (Pin_1); no longer J1.2 (Pin_2)
- net gnd.: now also J2.1 (Pin_1); no longer J2.2 (Pin_2)

Commit message: finally finished this
Parts:
- added D61, D62, D63, D64: LED, custom:pad - oval2.5x1.5, symbol Device:LED
Connections:
- net +: now also D61.1 (K), D61.2 (A)
- net +.: now also D63.1 (K), D63.2 (A)
- net gnd: now also D62.1 (K), D62.2 (A)
- net gnd.: now also D64.1 (K), D64.2 (A)
